File: receiver/receiver.sch (EAGLE design)
At the start: 10 parts, among them P1 PROMICRO_HEADER, P2 PROMICRO_HEADER, U1 CORE51822B, U2 AZ1117IH

Commit message: finish routing vias
Connections:
- removed net N$12: RA1.P$2, RA1.P$3
- new net N$2: RA1.P$3, RA1.P$4
- net LED-B: now also RA1.P$1; no longer RA1.P$4
- net LED-G: now also RA1.P$8; no longer RA1.P$7
- net LED-R: now also RA1.P$2; no longer RA1.P$1
- net N$10: now also RA1.P$7; no longer RA1.P$6
- net N$11: now also RA1.P$6; no longer RA1.P$5
- net N$14: now also RA1.P$5; no longer RA1.P$8
Changed lines of the file:
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@@
 <net name="LED-G" class="0">
-<segment>
-<pinref part="RA1" gate="G$1" pin="P$7"/>
-<wire x1="109.22" y1="53.34" x2="109.22" y2="43.18" width="0.1524" layer="91"/>
-<label x="106.68" y="40.64" size="1.778" layer="95"/>
-</segment>
 <segment>
 <pinref part="P1" gate="G$1" pin="P$5"/>
 <wire x1="10.16" y1="101.6" x2="27.94" y2="101.6" width="0.1524" layer="91"/>
 <label x="27.94" y="101.6" size="1.778" layer="95"/>
+</segment>
+<segment>
+<pinref part="RA1" gate="G$1" pin="P$8"/>
+<wire x1="114.3" y1="53.34" x2="114.3" y2="48.26" width="0.1524" layer="91"/>
+<wire x1="114.3" y1="48.26" x2="124.46" y2="48.26" width="0.1524" layer="91"/>
+<label x="124.46" y="48.26" size="1.778" layer="95"/>
 </segment>
 </net>
@@
 <pinref part="D1" gate="G$1" pin="RED(CATHODE)"/>
 <wire x1="111.76" y1="30.48" x2="99.06" y2="30.48" width="0.1524" layer="91"/>
-<pinref part="RA1" gate="G$1" pin="P$5"/>
-<wire x1="99.06" y1="30.48" x2="99.06" y2="53.34" width="0.1524" layer="91"/>
+<wire x1="99.06" y1="30.48" x2="99.06" y2="38.1" width="0.1524" layer="91"/>
+<wire x1="99.06" y1="38.1" x2="104.14" y2="38.1" width="0.1524" layer="91"/>
+<pinref part="RA1" gate="G$1" pin="P$6"/>
+<wire x1="104.14" y1="38.1" x2="104.14" y2="53.34" width="0.1524" layer="91"/>
 </segment>
 </net>
 <net name="N$10" class="0">
 <segment>
-<pinref part="RA1" gate="G$1" pin="P$6"/>
-<wire x1="104.14" y1="53.34" x2="104.14" y2="35.56" width="0.1524" layer="91"/>
-<wire x1="104.14" y1="35.56" x2="132.08" y2="35.56" width="0.1524" layer="91"/>
 <pinref part="D1" gate="G$1" pin="GREEN(CATHODE)"/>
-<wire x1="132.08" y1="35.56" x2="132.08" y2="30.48" width="0.1524" layer="91"/>
 <wire x1="132.08" y1="30.48" x2="127" y2="30.48" width="0.1524" layer="91"/>
-</segment>
-</net>
-<net name="N$12" class="0">
-<segment>
-<pinref part="RA1" gate="G$1" pin="P$2"/>
-<wire x1="104.14" y1="73.66" x2="104.14" y2="83.82" width="0.1524" layer="91"/>
-<wire x1="104.14" y1="83.82" x2="109.22" y2="83.82" width="0.1524" layer="91"/>
-<pinref part="RA1" gate="G$1" pin="P$3"/>
-<wire x1="109.22" y1="83.82" x2="109.22" y2="73.66" width="0.1524" layer="91"/>
+<wire x1="132.08" y1="30.48" x2="132.08" y2="45.72" width="0.1524" layer="91"/>
+<wire x1="132.08" y1="45.72" x2="109.22" y2="45.72" width="0.1524" layer="91"/>
+<pinref part="RA1" gate="G$1" pin="P$7"/>
+<wire x1="109.22" y1="45.72" x2="109.22" y2="53.34" width="0.1524" layer="91"/>
 </segment>
 </net>
@@
 <pinref part="D1" gate="G$1" pin="BLUE(CATHODE)"/>
 <wire x1="127" y1="25.4" x2="137.16" y2="25.4" width="0.1524" layer="91"/>
-<pinref part="RA1" gate="G$1" pin="P$8"/>
-<wire x1="137.16" y1="25.4" x2="137.16" y2="48.26" width="0.1524" layer="91"/>
-<wire x1="114.3" y1="53.34" x2="114.3" y2="48.26" width="0.1524" layer="91"/>
-<wire x1="114.3" y1="48.26" x2="137.16" y2="48.26" width="0.1524" layer="91"/>
+<wire x1="119.38" y1="20.32" x2="137.16" y2="20.32" width="0.1524" layer="91"/>
+<wire x1="137.16" y1="20.32" x2="137.16" y2="25.4" width="0.1524" layer="91"/>
+<wire x1="119.38" y1="20.32" x2="119.38" y2="7.62" width="0.1524" layer="91"/>
+<wire x1="119.38" y1="7.62" x2="96.52" y2="7.62" width="0.1524" layer="91"/>
+<wire x1="96.52" y1="7.62" x2="96.52" y2="53.34" width="0.1524" layer="91"/>
+<pinref part="RA1" gate="G$1" pin="P$5"/>
+<wire x1="96.52" y1="53.34" x2="99.06" y2="53.34" width="0.1524" layer="91"/>
 </segment>
 </net>
@@
 </segment>
 <segment>
-<pinref part="RA1" gate="G$1" pin="P$1"/>
-<wire x1="99.06" y1="88.9" x2="99.06" y2="73.66" width="0.1524" layer="91"/>
-<label x="96.52" y="88.9" size="1.778" layer="95"/>
+<pinref part="RA1" gate="G$1" pin="P$2"/>
+<wire x1="104.14" y1="73.66" x2="104.14" y2="88.9" width="0.1524" layer="91"/>
+<label x="104.14" y="88.9" size="1.778" layer="95" rot="R90"/>
 </segment>
 </net>
@@
 </segment>
 <segment>
-<pinref part="RA1" gate="G$1" pin="P$4"/>
-<wire x1="114.3" y1="73.66" x2="114.3" y2="88.9" width="0.1524" layer="91"/>
-<label x="111.76" y="88.9" size="1.778" layer="95"/>
+<pinref part="RA1" gate="G$1" pin="P$1"/>
+<wire x1="99.06" y1="88.9" x2="99.06" y2="73.66" width="0.1524" layer="91"/>
+<label x="99.06" y="88.9" size="1.778" layer="95" rot="R90"/>
 </segment>
 </net>
@@
 </segment>
 </net>
+<net name="N$2" class="0">
+<segment>
+<pinref part="RA1" gate="G$1" pin="P$3"/>
+<wire x1="109.22" y1="73.66" x2="109.22" y2="81.28" width="0.1524" layer="91"/>
+<wire x1="109.22" y1="81.28" x2="114.3" y2="81.28" width="0.1524" layer="91"/>
+<pinref part="RA1" gate="G$1" pin="P$4"/>
+<wire x1="114.3" y1="81.28" x2="114.3" y2="73.66" width="0.1524" layer="91"/>
+</segment>
+</net>

Commit message: update drill size to 10mil
Changed lines of the file:
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@@
 </variantdefs>
 <classes>
-<class number="0" name="default" width="0.3048" drill="0.508">
+<class number="0" name="default" width="0.3048" drill="0.254">
 <clearance class="0" value="0.254"/>
 </class>
@@
 <instance part="GND3" gate="1" x="-20.32" y="76.2"/>
 <instance part="GND4" gate="1" x="30.48" y="109.22" rot="R90"/>
-<instance part="P+1" gate="VCC" x="119.38" y="109.22" rot="R90"/>
+<instance part="P+1" gate="VCC" x="129.54" y="101.6" rot="R90"/>
 <instance part="D1" gate="G$1" x="119.38" y="27.94"/>
 <instance part="RA2" gate="G$1" x="71.12" y="-2.54"/>
@@
 <pinref part="U2" gate="G$1" pin="VOUT"/>
 <pinref part="P+1" gate="VCC" pin="VCC"/>
-<wire x1="137.16" y1="109.22" x2="121.92" y2="109.22" width="0.1524" layer="91"/>
+<wire x1="137.16" y1="109.22" x2="132.08" y2="101.6" width="0.1524" layer="91"/>
 <pinref part="U2" gate="G$1" pin="OUTPUT"/>
-<wire x1="142.24" y1="109.22" x2="121.92" y2="109.22" width="0.1524" layer="91"/>
-<junction x="121.92" y="109.22"/>
+<wire x1="142.24" y1="109.22" x2="132.08" y2="101.6" width="0.1524" layer="91"/>
+<junction x="132.08" y="101.6"/>
 </segment>
 <segment>
