File: numpad/numpad.brd (EAGLE design)
At the start: 100 x 100 mm, 22 parts

Commit message: update numpad
Parts:
- moved U$22 68.1 mm to (96.4, 29.8), turned to 180 degrees
- moved U$1 45.9 mm to (88.2, 14.2), turned to 180 degrees
- moved U$21 3.20 mm to (68.0, 12.5)
- moved U$20 2.92 mm to (48.5, 12.5)
- moved U$17 2.83 mm to (68.0, 32.0)
- moved U$19 2.69 mm to (29.0, 12.5)
- moved U$18 2.55 mm to (9.50, 12.5)
- moved U$13 2.50 mm to (68.0, 51.5)
- moved U$16 2.50 mm to (48.5, 32.0)
- moved U$15 2.24 mm to (29.0, 32.0)
- moved U$9 2.24 mm to (68.0, 71.0)
- moved U$12 2.12 mm to (48.5, 51.5)
- moved U$14 2.06 mm to (9.50, 32.0)
- moved U$5 2.06 mm to (68.0, 90.5)
- moved U$11 1.80 mm to (29.0, 51.5)
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Routing:
- net B$1: track 0.00 -> 400.5 mm
- net P0: track 0.00 -> 159.6 mm
- net P1: track 0.00 -> 118.1 mm, vias 0 -> 1
- net P4: track 0.00 -> 113.0 mm, vias 0 -> 1
- net P2: track 0.00 -> 94.5 mm, vias 0 -> 1
- net P5: track 0.00 -> 93.4 mm, vias 0 -> 1
- net P8: track 0.00 -> 91.7 mm, vias 0 -> 1
- net P6: track 0.00 -> 87.9 mm
- net P9: track 0.00 -> 87.1 mm
- net P3: track 0.00 -> 85.0 mm
- net P12: track 0.00 -> 80.4 mm, vias 0 -> 1
- net P16: track 0.00 -> 77.4 mm, vias 0 -> 1
- net P10: track 0.00 -> 66.6 mm
- net P7: track 0.00 -> 63.6 mm
- net P17: track 0.00 -> 62.9 mm
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